File: tessel-raspi-b-plus.brd (EAGLE design)
At the start: 87.1 x 55.9 mm, 3 parts, among them J1 MODULE_HEADER_MODULEDEFAULT, J2 MODULE_HEADER_MODULEDEFAULT

Commit message: added silkscreen text
fixed repo

Create README.md
Parts:
- moved J2 35.3 mm to (63.5, 54.0)
- moved J1 25.7 mm to (33.0, 54.0)
- moved JP1 22.1 mm to (54.6, 3.50)
Routing:
- net TX: track 91.9 -> 49.7 mm
- net RX: track 91.6 -> 49.7 mm
- net GPIO_1_3: track 90.4 -> 49.7 mm
- net GPIO_2_3: track 57.3 -> 62.8 mm
- net GPIO_2_2: track 57.3 -> 62.8 mm
- net GPIO_2_1: track 57.3 -> 62.8 mm
- net SCK: track 89.7 -> 86.1 mm, vias 2 -> 1
- net MISO: track 88.1 -> 91.4 mm
- net SDA: track 89.8 -> 88.2 mm
- net SCL: track 87.0 -> 85.5 mm, vias 2 -> 1
- net MOSI: track 87.2 -> 87.7 mm, vias 2 -> 1
Other:
- board outline removed
- board text added: "/Users/nlintz/Desktop/bw_bmp/hexagon_bw.bmp"
- board text added: "PTP-Adapter"
- board text added: "Raspberry Pi B+"
- board text added: "Revision 0.0"
